File: Coral_stepper_controller/Stepper_Motor_module_V1/_autosave-Motor_module.kicad_sch (KiCad schematic)
At the start: 34 parts, among them J1 Limit Switch, J2 Limit Switch, J3 Limit Switch, J4 Limit Switch, J5 Conn_01x08_Male, J6 Conn_01x04_Male, J7 Conn_01x08_Female, J8 Conn_01x08_Female, SW1 SW_Push, U1 STM32F031F6P6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

Commit message: udated by FZ
Parts:
- U1: value STM32F031F6P6 -> (none)
Changed lines of the file:
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@@
       (effects (font (size 1.27 1.27)) (justify left))
     )
-    (property "Value" "STM32F031F6P6" (id 1) (at 49.53 57.15 90)
+    (property "Value" "" (id 1) (at 49.53 57.15 90)
       (effects (font (size 1.27 1.27)) (justify left))
     )
