File: Coral_stepper_controller/Stepper_Motor_module_V1/Motor_module.kicad_pcb (KiCad board)
At the start: 2 copper layers, 28.5 x 40 mm, 34 parts, among them J1 Limit Switch, J2 Limit Switch, J3 Limit Switch, J4 Limit Switch, J5 Conn_01x08_Male, J6 Conn_01x04_Male, J7 Conn_01x08_Female, J8 Conn_01x08_Female, SW1 SW_Push, U1 STM32F031F6Px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

Commit message: udated by FZ
Parts:
- U1: value STM32F031F6Px -> STM32F031F6P6
Routing:
- net /SWCLK: track 45.7 -> 44.9 mm
- net /RS485_DE: track 14.6 -> 13.9 mm
